Commit message: feat: add Jazzy support

File: khi_description/urdf/bx/khi.ros2_control.xacro (robot description, xacro)
@@ -7,4 +7,5 @@
     simulation
     use_gazebo
+    use_gz
     robot_ip
     robot_controller
@@ -19,5 +20,6 @@
     ft_sensor
     ">
-    <ros2_control name="${robot_name}" type="system">
+    <xacro:property name="safe_robot_name" value="${robot_name.replace('-', '_')}" />
+    <ros2_control name="${safe_robot_name}" type="system">
       <xacro:include filename="$(find khi_description)/urdf/$(arg robot_series)/get_mechanical_parameters.xacro"/>
       <xacro:include filename="$(find khi_description)/urdf/$(arg robot_series)/get_joint_limits.xacro"/>
@@ -30,5 +32,8 @@
           <plugin>gazebo_ros2_control/GazeboSystem</plugin>
         </xacro:if>
-        <xacro:unless value="${use_gazebo}">
+        <xacro:if value="${use_gz}">
+          <plugin>gz_ros2_control/GazeboSimSystem</plugin>
+        </xacro:if>
+        <xacro:unless value="${use_gazebo or use_gz}">
           <plugin>khi_hardware/KhiHardwareInterface</plugin>
           <param name="robot_name">$(arg robot_name)</param>
@@ -113,5 +118,5 @@
         <param name="arm">arm1</param>
       </joint>
-      <xacro:if value="${use_gazebo}">
+      <xacro:if value="${use_gazebo or use_gz}">
         <xacro:if value="${is_parallel}">
           <joint name="${prefix}parallel_joint1">

File: khi_description/urdf/rs/khi.ros2_control.xacro (robot description, xacro)
@@ -7,4 +7,5 @@
     simulation
     use_gazebo
+    use_gz
     robot_ip
     robot_controller
@@ -19,5 +20,6 @@
     ft_sensor
     ">
-    <ros2_control name="${robot_name}" type="system">
+    <xacro:property name="safe_robot_name" value="${robot_name.replace('-', '_')}" />
+    <ros2_control name="${safe_robot_name}" type="system">
       <xacro:include filename="$(find khi_description)/urdf/$(arg robot_series)/get_mechanical_parameters.xacro"/>
       <xacro:include filename="$(find khi_description)/urdf/$(arg robot_series)/get_joint_limits.xacro"/>
@@ -30,5 +32,8 @@
           <plugin>gazebo_ros2_control/GazeboSystem</plugin>
         </xacro:if>
-        <xacro:unless value="${use_gazebo}">
+        <xacro:if value="${use_gz}">
+          <plugin>gz_ros2_control/GazeboSimSystem</plugin>
+        </xacro:if>
+        <xacro:unless value="${use_gazebo or use_gz}">
           <plugin>khi_hardware/KhiHardwareInterface</plugin>
           <param name="robot_name">$(arg robot_name)</param>

File: khi_description/urdf/wd/khi.ros2_control.xacro (robot description, xacro)
@@ -7,4 +7,5 @@
     simulation
     use_gazebo
+    use_gz
     robot_ip
     robot_controller
@@ -19,5 +20,6 @@
     ft_sensor
     ">
-    <ros2_control name="${robot_name}" type="system">
+    <xacro:property name="safe_robot_name" value="${robot_name.replace('-', '_')}" />
+    <ros2_control name="${safe_robot_name}" type="system">
       <xacro:include filename="$(find khi_description)/urdf/$(arg robot_series)/get_mechanical_parameters.xacro"/>
       <xacro:include filename="$(find khi_description)/urdf/$(arg robot_series)/get_joint_limits.xacro"/>
@@ -31,5 +33,8 @@
           <plugin>gazebo_ros2_control/GazeboSystem</plugin>
         </xacro:if>
-        <xacro:unless value="${use_gazebo}">
+        <xacro:if value="${use_gz}">
+          <plugin>gz_ros2_control/GazeboSimSystem</plugin>
+        </xacro:if>
+        <xacro:unless value="${use_gazebo or use_gz}">
           <plugin>khi_hardware/KhiHardwareInterface</plugin>
           <param name="robot_name">$(arg robot_name)</param>
@@ -152,5 +157,5 @@
         <param name="arm">arm2</param>
       </joint>
-      <xacro:if value="${use_gazebo}">
+      <xacro:if value="${use_gazebo or use_gz}">
         <joint name="${prefix}lower_joint3_mimic1">
           <param name="type"> ${lower_jt3_mimic1_type} </param>
